Commit message: v0.0.6

File: packages/install/uwaba_prototype_description/share/uwaba_prototype_description/urdf/uwaba_prototype_misplaced_sup.urdf (robot description, URDF)
Before this commit: robot uwaba_prototype, 30 links, 29 joints
Links:
- removed link laser_frame
- added link scan_link, mass 0.2500000000; collision cylinder length=0.0183099993 radius=0.0341599993; visual cylinder length=0.0183099993 radius=0.0341599993
- link Left_bumped_treads_link: geometry collision mesh filename=package://uwaba_prototype_description/meshes/dae/right.trac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 scale=1.0000000000 1.0000000000 1.0000000000; visual mesh filename=package://uwaba_prototype_description/meshes/dae/right.trac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 scale=1.0000000000 1.0000000000 1.0000000000
- link Left_small_wheels_frame.001_link: mass 0.0500000007 -> 0.0099999998
- link Left_small_wheels_frame.002_link: mass 0.0500000007 -> 0.0099999998
- link Left_small_wheels_frame.003_link: mass 0.0500000007 -> 0.0099999998
- link Left_small_wheels_frame.004_link: mass 0.0500000007 -> 0.0099999998
- link Left_small_wheels_frame_link: mass 0.0500000007 -> 0.0099999998
- link Left_wheel.001_link: mass 0.1000000015 -> 0.0500000007
- link Left_wheel.002_link: mass 0.1000000015 -> 0.0500000007
- link Left_wheel.003_link: mass 0.1000000015 -> 0.0500000007
- link Left_wheel.004_link: mass 0.1000000015 -> 0.0500000007
- link Left_wheel.005_link: mass 0.1000000015 -> 0.0500000007
- link Left_wheel.006_link: mass 0.1000000015 -> 0.0750000030
- link Left_wheel_sprocket_link: mass 0.1000000015 -> 0.0750000030
- link Right_bumped_treads_link: geometry collision mesh filename=package://uwaba_prototype_description/meshes/dae/left.track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 scale=1.0000000000 1.0000000000 1.0000000000; visual mesh filename=package://uwaba_prototype_description/meshes/dae/left.track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 scale=1.0000000000 1.0000000000 1.0000000000
- link Right_small_wheels_frame.001_link: mass 0.0500000007 -> 0.0099999998
- link Right_small_wheels_frame.002_link: mass 0.0500000007 -> 0.0099999998
- link Right_small_wheels_frame.003_link: mass 0.0500000007 -> 0.0099999998
- link Right_small_wheels_frame.004_link: mass 0.0500000007 -> 0.0099999998
- link Right_small_wheels_frame_link: mass 0.0500000007 -> 0.0099999998
- link Right_wheel.001_link: mass 0.1000000015 -> 0.0500000007
- link Right_wheel.002_link: mass 0.1000000015 -> 0.0500000007
- link Right_wheel.003_link: mass 0.1000000015 -> 0.0500000007
- link Right_wheel.004_link: mass 0.1000000015 -> 0.0500000007
- link Right_wheel.005_link: mass 0.1000000015 -> 0.0500000007
- link Right_wheel.006_link: mass 0.1000000015 -> 0.0750000030
- link Right_wheel_sprocket_link: mass 0.1000000015 -> 0.0750000030
- link base_link: mass 1.2999999523 -> 1.0000000000
- link support_link: mass None -> 0.1500000060; geometry collision mesh filename=package://uwaba_prototype_description/meshes/dae/Cube.002.d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 scale=1.0000000000 1.0000000000 1.0000000000; visual box size=0.2480000257 0.1058000028 0.0357334018
Joints:
- removed joint Left_sprocket_base_joint
- removed joint Left_suspension.001_base_joint
- removed joint Left_suspension.002_base_joint
- removed joint Left_suspension.003_base_joint
- removed joint Left_suspension.004_base_joint
- removed joint Left_suspension_base_joint
- removed joint Left_tracks_base_joint
- removed joint Left_wheel.001_suspension_joint
- removed joint Left_wheel.002_suspension_joint
- removed joint Left_wheel.003_suspension_joint
- removed joint Left_wheel.004_suspension_joint
- removed joint Left_wheel.005_suspension_joint
- removed joint Left_wheel.006_base_joint
- removed joint Right_sprocket_base_joint
- removed joint Right_suspension.001_base_joint
- removed joint Right_suspension.002_base_joint
- removed joint Right_suspension.003_base_joint
- removed joint Right_suspension.004_base_joint
- removed joint Right_suspension_base_joint
- removed joint Right_tracks_base_joint
- removed joint Right_wheel.001_suspension_joint
- removed joint Right_wheel.002_suspension_joint
- removed joint Right_wheel.003_suspension_joint
- removed joint Right_wheel.004_suspension_joint
- removed joint Right_wheel.005_suspension_joint
- removed joint Right_wheel.006_base_joint
- removed joint laser_frame_base_joint
- removed joint supprot_base_joint
- added joint left_bumped_thread_base_joint: type fixed, parent base_link, child Left_bumped_treads_link, origin xyz=-0.0000073090 0.0762520012 -0.0125610121 rpy=0.0000000000 0.0000000000 0.0000000000
- added joint left_sprocket_base_joint: type continuous, parent base_link, child Left_wheel_sprocket_link, origin xyz=-0.1065520449 0.0762500119 0.0002469979 rpy=0.0000000000 0.0000000000 0.0000000000, axis 0.0000000000 1.0000000000 0.0000000000, limit lower=0 upper=0 effort=0.0000000000 velocity=0.0000000000
- added joint left_suspension.001_base_joint: type revolute, parent base_link, child Left_small_wheels_frame.001_link, origin xyz=0.0515604214 0.0552990314 -0.0151900463 rpy=0.0000000000 0.0000000000 0.0000000000, axis 0.0000000000 1.0000000000 0.0000000000, limit lower=-0.1745329946 upper=0.1745329946 effort=0.0000000000 velocity=0.0000000000
- added joint left_suspension.002_base_joint: type revolute, parent base_link, child Left_small_wheels_frame.002_link, origin xyz=0.0197104206 0.0552989979 -0.0151902959 rpy=0.0000000000 0.0000000000 0.0000000000, axis 0.0000000000 1.0000000000 0.0000000000, limit lower=-0.1745329946 upper=0.1745329946 effort=0.0000000000 velocity=0.0000000000
- added joint left_suspension.003_base_joint: type revolute, parent base_link, child Left_small_wheels_frame.003_link, origin xyz=-0.0153435795 0.0552989904 -0.0151902996 rpy=0.0000000000 0.0000000000 0.0000000000, axis 0.0000000000 1.0000000000 0.0000000000, limit lower=-0.1745329946 upper=0.1745329946 effort=0.0000000000 velocity=0.0000000000
- added joint left_suspension.004_base_joint: type revolute, parent base_link, child Left_small_wheels_frame.004_link, origin xyz=-0.0490785828 0.0552990314 -0.0151903071 rpy=0.0000000000 0.0000000000 0.0000000000, axis 0.0000000000 1.0000000000 0.0000000000, limit lower=-0.1745329946 upper=0.1745329946 effort=0.0000000000 velocity=0.0000000000
- added joint left_suspension_base_joint: type revolute, parent base_link, child Left_small_wheels_frame_link, origin xyz=0.0879334183 0.0552990426 -0.0151902996 rpy=0.0000000000 0.0000000000 0.0000000000, axis 0.0000000000 1.0000000000 0.0000000000, limit lower=-0.1745329946 upper=0.1745329946 effort=0.0000000000 velocity=0.0000000000
- added joint left_wheel.001_suspension_joint: type fixed, parent Left_small_wheels_frame.004_link, child Left_wheel.001_link, origin xyz=-0.0191554390 0.0209509283 -0.0199896954 rpy=-0.0000000000 0.0000000000 0.0000000000
- added joint left_wheel.002_suspension_joint: type fixed, parent Left_small_wheels_frame.003_link, child Left_wheel.002_link, origin xyz=-0.0184964389 0.0209509470 -0.0199897066 rpy=-0.0000000000 0.0000000000 0.0000000000
- added joint left_wheel.003_suspension_joint: type fixed, parent Left_small_wheels_frame.002_link, child Left_wheel.003_link, origin xyz=-0.0197104495 0.0209509693 -0.0199897159 rpy=-0.0000000000 0.0000000000 0.0000000000
- added joint left_wheel.004_suspension_joint: type fixed, parent Left_small_wheels_frame.001_link, child Left_wheel.004_link, origin xyz=-0.0179914646 0.0209509209 -0.0199899562 rpy=-0.0000000000 0.0000000000 0.0000000000
- added joint left_wheel.005_suspension_joint: type fixed, parent Left_small_wheels_frame_link, child Left_wheel.005_link, origin xyz=-0.0192444250 0.0209509395 -0.0199897159 rpy=-0.0000000000 0.0000000000 0.0000000000
- added joint left_wheel.006_base_joint: type fixed, parent base_link, child Left_wheel.006_link, origin xyz=0.1065519945 0.0762500119 0.0002470016 rpy=0.0000000000 0.0000000000 0.0000000000
- added joint right_bumped_thread_base_joint: type fixed, parent base_link, child Right_bumped_treads_link, origin xyz=0.0000440089 -0.0765780109 -0.0125610270 rpy=0.0000000000 0.0000000000 0.0000000000
- added joint right_sprocket_base_joint: type continuous, parent base_link, child Right_wheel_sprocket_link, origin xyz=-0.1065520300 -0.0762500215 0.0002470128 rpy=0.0000000000 0.0000000000 0.0000000000, axis 0.0000000000 1.0000000000 0.0000000000, limit lower=0 upper=0 effort=0.0000000000 velocity=0.0000000000
- added joint right_suspension.001_base_joint: type revolute, parent base_link, child Right_small_wheels_frame.001_link, origin xyz=0.0515604140 -0.0552989628 -0.0151902884 rpy=0.0000000000 0.0000000000 0.0000000000, axis 0.0000000000 1.0000000000 0.0000000000, limit lower=-0.1745329946 upper=0.1745329946 effort=0.0000000000 velocity=0.0000000000
- added joint right_suspension.002_base_joint: type revolute, parent base_link, child Right_small_wheels_frame.002_link, origin xyz=0.0197104187 -0.0552990224 -0.0151902996 rpy=0.0000000000 0.0000000000 0.0000000000, axis 0.0000000000 1.0000000000 0.0000000000, limit lower=-0.1745329946 upper=0.1745329946 effort=0.0000000000 velocity=0.0000000000
- added joint right_suspension.003_base_joint: type revolute, parent base_link, child Right_small_wheels_frame.003_link, origin xyz=-0.0153435786 -0.0552990075 -0.0151903033 rpy=0.0000000000 0.0000000000 0.0000000000, axis 0.0000000000 1.0000000000 0.0000000000, limit lower=-0.1745329946 upper=0.1745329946 effort=0.0000000000 velocity=0.0000000000
- added joint right_suspension.004_base_joint: type revolute, parent base_link, child Right_small_wheels_frame.004_link, origin xyz=-0.0490785791 -0.0552989665 -0.0151903071 rpy=0.0000000000 0.0000000000 0.0000000000, axis 0.0000000000 1.0000000000 0.0000000000, limit lower=-0.1745329946 upper=0.1745329946 effort=0.0000000000 velocity=0.0000000000
- added joint right_suspension_base_joint: type revolute, parent base_link, child Right_small_wheels_frame_link, origin xyz=0.0879334183 -0.0552989665 -0.0151903033 rpy=0.0000000000 0.0000000000 0.0000000000, axis 0.0000000000 1.0000000000 0.0000000000, limit lower=-0.1745329946 upper=0.1745329946 effort=0.0000000000 velocity=0.0000000000
- added joint right_wheel.001_suspension_joint: type fixed, parent Right_small_wheels_frame.004_link, child Right_wheel.001_link, origin xyz=-0.0191554353 -0.0209510326 -0.0199897029 rpy=0.0000000000 0.0000000000 0.0000000000
- added joint right_wheel.002_suspension_joint: type fixed, parent Right_small_wheels_frame.003_link, child Right_wheel.002_link, origin xyz=-0.0184964174 -0.0209510289 -0.0199897103 rpy=0.0000000000 0.0000000000 0.0000000000
- added joint right_wheel.003_suspension_joint: type fixed, parent Right_small_wheels_frame.002_link, child Right_wheel.003_link, origin xyz=-0.0197104261 -0.0209509619 -0.0199897196 rpy=0.0000000000 0.0000000000 0.0000000000
- added joint right_wheel.004_suspension_joint: type fixed, parent Right_small_wheels_frame.001_link, child Right_wheel.004_link, origin xyz=-0.0179914236 -0.0209510438 -0.0199897178 rpy=0.0000000000 0.0000000000 0.0000000000
- added joint right_wheel.005_suspension_joint: type fixed, parent Right_small_wheels_frame_link, child Right_wheel.005_link, origin xyz=-0.0192444548 -0.0209510252 -0.0199896898 rpy=0.0000000000 0.0000000000 0.0000000000
- added joint right_wheel.006_base_joint: type fixed, parent base_link, child Right_wheel.006_link, origin xyz=0.1065519945 -0.0762500066 0.0002470054 rpy=0.0000000000 0.0000000000 0.0000000000
- added joint scan_base_joint: type fixed, parent base_link, child scan_link, origin xyz=-0.0110695819 -0.0000000043 0.0737789795 rpy=0.0000000000 0.0000000000 0.0000000000
- added joint support_base_joint: type fixed, parent base_link, child support_link, origin xyz=0.0000000177 0.0000000048 0.0524450019 rpy=0.0000000000 0.0000000000 0.0000000000

File: packages/src/uwaba_prototype_description/urdf/uwaba_prototype-bkup.urdf (robot description, URDF)
Before this commit: robot uwaba_prototype, 30 links, 29 joints
Links:
- removed link laser_frame
- added link scan_link, mass 0.3000000119; collision cylinder length=0.0183099993 radius=0.0341599993; visual cylinder length=0.0183099993 radius=0.0341599993
- link Left_bumped_treads_link: geometry collision mesh filename=package://uwaba_prototype_description/meshes/dae/right.trac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 scale=1.0000000000 1.0000000000 1.0000000000; visual mesh filename=package://uwaba_prototype_description/meshes/dae/right.trac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 scale=1.0000000000 1.0000000000 1.0000000000
- link Right_bumped_treads_link: geometry collision mesh filename=package://uwaba_prototype_description/meshes/dae/left.track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 scale=1.0000000000 1.0000000000 1.0000000000; visual mesh filename=package://uwaba_prototype_description/meshes/dae/left.track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 scale=1.0000000000 1.0000000000 1.0000000000
- link support_link: geometry collision mesh filename=package://uwaba_prototype_description/meshes/dae/Cube.002.d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 scale=0.9999999404 0.9999999404 0.9999898076; visual mesh filename=package://uwaba_prototype_description/meshes/dae/Cube.002.d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 scale=0.9999999404 0.9999999404 0.9999898076
Joints:
- removed joint laser_frame_base_joint
- added joint scan_base_joint: type fixed, parent base_link, child scan_link, origin xyz=-0.0110695819 -0.0000000043 0.0737789795 rpy=0.0000000000 0.0000000000 0.0000000000

File: packages/src/uwaba_prototype_nav2/description/uwaba_prototype_nav2_plugins.xacro (robot description, xacro)
@@ -1,3 +1,4 @@
 <robot name="uwaba_prototype_nav2_plugins" version="1.0"
     xmlns:xacro="http://www.ros.org/wiki/xacro">
+    <!-- ... -->
 </robot>
