Commit message: v0.0.12

File: packages/src/uwaba_prototype_diffbot/description/ros2_control/diffbot.ros2_control.xacro (robot description, xacro)
@@ -5,5 +5,5 @@
       <xacro:unless value="${use_mock_hardware}">
         <hardware>
-          <plugin>ros2_control_demo_example_2/DiffBotSystemHardware</plugin>
+          <plugin>uwaba_prototype_diffbot/DiffBotSystemHardware</plugin>
           <param name="example_param_hw_start_duration_sec">0</param>
           <param name="example_param_hw_stop_duration_sec">3.0</param>
@@ -16,13 +16,13 @@
         </hardware>
       </xacro:if>
-      <joint name="${prefix}left_wheel_joint">
-        <command_interface name="velocity"/>
-        <state_interface name="position"/>
-        <state_interface name="velocity"/>
+      <joint name="Left_sprocket_base_joint">
+        <command_interface name="velocity" />
+        <state_interface name="position" />
+        <state_interface name="velocity" />
       </joint>
-      <joint name="${prefix}right_wheel_joint">
-        <command_interface name="velocity"/>
-        <state_interface name="position"/>
-        <state_interface name="velocity"/>
+      <joint name="Right_sprocket_base_joint">
+        <command_interface name="velocity" />
+        <state_interface name="position" />
+        <state_interface name="velocity" />
       </joint>
     </ros2_control>
