Commit message: v0.0.29

File: packages/src/uwaba_prototype_description/urdf/uwaba_prototype-with-prefixes.urdf.xacro (robot description, xacro)
@@ -2,4 +2,5 @@
 <robot name="uwaba_prototype_diffbot" version="1.0"
   xmlns:xacro="http://www.ros.org/wiki/xacro">
+  <xacro:macro name="diffbot" params="prefix">
   <material name="wheels-grey">
     <color rgba="0.25 0.25 0.25 1.00000" />
@@ -904,3 +905,4 @@
     </visual>
   </link>
+</xacro:macro>
 </robot>
