Commit message: v0.14.0

File: packages/src/uwaba_prototype_description/urdf/uwaba_prototype.urdf.xacro (robot description, xacro)
@@ -210,4 +210,16 @@
     <child link="base_link" />
   </joint>
+  <!-- <joint name="imu_base_joint" type="fixed">
+    <origin rpy="0.0000000000 0.0000000000 0.0000000000"
+      xyz="0.182000041 0.054800018 0.02375" />
+    <parent link="base_link" />
+    <child link="imu_frame" />
+  </joint> -->
+  <joint name="imu_base_joint" type="fixed">
+    <origin rpy="0.0000000000 0.0000000000 0.0000000000"
+      xyz="0.061 -0.004 0.001875" />
+    <parent link="base_link" />
+    <child link="imu_frame" />
+  </joint>
   <joint name="laser_frame_base_joint" type="fixed">
     <origin rpy="0.0000000000 0.0000000000 0.0000000000"
@@ -837,4 +849,21 @@
   </link>
   <link name="base_footprint" />
+  <link name="imu_frame">
+    <collision name="imu_collision">
+      <origin rpy="0.0000000000 0.0000000000 0.0000000000"
+        xyz="0 0 0" />
+      <geometry>
+        <box size="0.001 0.002 0.001" />
+      </geometry>
+    </collision>
+    <visual>
+      <!-- <material name="base-blue" /> -->
+      <origin rpy="0.0000000000 0.0000000000 0.0000000000"
+        xyz="0 0 0" />
+      <geometry>
+        <box size="0.001 0.002 0.001" />
+      </geometry>
+    </visual>
+  </link>
   <link name="base_link">
     <collision name="base_collision">

Commit message: v0.16.0

File: packages/src/uwaba_prototype_description/urdf/uwaba_prototype.urdf.xacro (robot description, xacro)
@@ -892,5 +892,5 @@
   <link name="laser_frame">
     <collision name="laser_frame_collision">
-      <origin rpy="0.0000000000 0.0000000000 0.0000000000"
+      <origin rpy="0.0000000000 3.14159265359 0.0000000000"
         xyz="0.0000000000 -0.0000000000 0.0000000000" />
       <geometry>
@@ -901,9 +901,9 @@
       <inertia ixx="0.0000958993" ixy="0.0000000000" ixz="0.0000000000" iyy="0.0000958993"
         iyz="0.0000000000" izz="0.0001750358" />
-      <origin rpy="0.0000000000 0.0000000000 0.0000000000"
+      <origin rpy="0.0000000000 3.14159265359 0.0000000000"
         xyz="0.0000000000 -0.0000000000 0.0000000000" />
       <mass value="0.3000000119" />
     </inertial>
-    <visual name="laser">
+    <visual>
       <material name="lidar-darkgrey" />
       <origin rpy="0.0000000000 0.0000000000 0.0000000000"

Commit message: v0.17.1

File: packages/src/uwaba_prototype_description/urdf/uwaba_prototype.urdf.xacro (robot description, xacro)
@@ -223,5 +223,5 @@
   </joint>
   <joint name="laser_frame_base_joint" type="fixed">
-    <origin rpy="0.0000000000 0.0000000000 0.0000000000"
+    <origin rpy="${pi} 0.0000000000 0.0000000000"
       xyz="-0.0110695819 -0.0000000043 0.0737789795" />
     <parent link="base_link" />
@@ -892,5 +892,5 @@
   <link name="laser_frame">
     <collision name="laser_frame_collision">
-      <origin rpy="0.0000000000 3.14159265359 0.0000000000"
+      <origin rpy="0.0000000000 0.0000000000 0.0000000000"
         xyz="0.0000000000 -0.0000000000 0.0000000000" />
       <geometry>
@@ -901,5 +901,5 @@
       <inertia ixx="0.0000958993" ixy="0.0000000000" ixz="0.0000000000" iyy="0.0000958993"
         iyz="0.0000000000" izz="0.0001750358" />
-      <origin rpy="0.0000000000 3.14159265359 0.0000000000"
+      <origin rpy="0.0000000000 0.0000000000 0.0000000000"
         xyz="0.0000000000 -0.0000000000 0.0000000000" />
       <mass value="0.3000000119" />

Commit message: v0.17.2

File: packages/src/uwaba_prototype_description/urdf/uwaba_prototype.urdf.xacro (robot description, xacro)
@@ -223,8 +223,9 @@
   </joint>
   <joint name="laser_frame_base_joint" type="fixed">
-    <origin rpy="${pi} 0.0000000000 0.0000000000"
+    <origin rpy="0.0000000000 0.0000000000 0.0000000000"
       xyz="-0.0110695819 -0.0000000043 0.0737789795" />
     <parent link="base_link" />
     <child link="laser_frame" />
+    <axis xyz="1.0000000000 0.0000000000 0.0000000000" />
   </joint>
   <joint name="support_base_joint" type="fixed">
@@ -892,5 +893,5 @@
   <link name="laser_frame">
     <collision name="laser_frame_collision">
-      <origin rpy="0.0000000000 0.0000000000 0.0000000000"
+      <origin rpy="${pi} 0.0000000000 0.0000000000"
         xyz="0.0000000000 -0.0000000000 0.0000000000" />
       <geometry>
@@ -901,5 +902,5 @@
       <inertia ixx="0.0000958993" ixy="0.0000000000" ixz="0.0000000000" iyy="0.0000958993"
         iyz="0.0000000000" izz="0.0001750358" />
-      <origin rpy="0.0000000000 0.0000000000 0.0000000000"
+      <origin rpy="${pi} 0.0000000000 0.0000000000"
         xyz="0.0000000000 -0.0000000000 0.0000000000" />
       <mass value="0.3000000119" />
@@ -907,5 +908,5 @@
     <visual>
       <material name="lidar-darkgrey" />
-      <origin rpy="0.0000000000 0.0000000000 0.0000000000"
+      <origin rpy="${pi} 0.0000000000 0.0000000000"
         xyz="0.0000000000 -0.0000000000 0.0000000000" />
       <geometry>

Commit message: 0.17.3

File: packages/src/uwaba_prototype_description/urdf/uwaba_prototype.urdf.xacro (robot description, xacro)
@@ -210,18 +210,12 @@
     <child link="base_link" />
   </joint>
-  <!-- <joint name="imu_base_joint" type="fixed">
-    <origin rpy="0.0000000000 0.0000000000 0.0000000000"
-      xyz="0.182000041 0.054800018 0.02375" />
+  <joint name="imu_base_joint" type="fixed">
+    <origin rpy="0.0000000000 0.0000000000 0.0000000000"
+      xyz="0.061 -0.004 0.001875" />
     <parent link="base_link" />
     <child link="imu_frame" />
-  </joint> -->
-  <joint name="imu_base_joint" type="fixed">
-    <origin rpy="0.0000000000 0.0000000000 0.0000000000"
-      xyz="0.061 -0.004 0.001875" />
-    <parent link="base_link" />
-    <child link="imu_frame" />
   </joint>
   <joint name="laser_frame_base_joint" type="fixed">
-    <origin rpy="0.0000000000 0.0000000000 0.0000000000"
+    <origin rpy="${pi} 0.0000000000 0.0000000000"
       xyz="-0.0110695819 -0.0000000043 0.0737789795" />
     <parent link="base_link" />

Commit message: v0.19.0

File: packages/src/uwaba_prototype_description/urdf/uwaba_prototype.urdf.xacro (robot description, xacro)
@@ -221,5 +221,4 @@
     <parent link="base_link" />
     <child link="laser_frame" />
-    <axis xyz="1.0000000000 0.0000000000 0.0000000000" />
   </joint>
   <joint name="support_base_joint" type="fixed">
@@ -887,5 +886,5 @@
   <link name="laser_frame">
     <collision name="laser_frame_collision">
-      <origin rpy="${pi} 0.0000000000 0.0000000000"
+      <origin rpy="0.0000000000 0.0000000000 0.0000000000"
         xyz="0.0000000000 -0.0000000000 0.0000000000" />
       <geometry>
@@ -896,5 +895,5 @@
       <inertia ixx="0.0000958993" ixy="0.0000000000" ixz="0.0000000000" iyy="0.0000958993"
         iyz="0.0000000000" izz="0.0001750358" />
-      <origin rpy="${pi} 0.0000000000 0.0000000000"
+      <origin rpy="0.0000000000 0.0000000000 0.0000000000"
         xyz="0.0000000000 -0.0000000000 0.0000000000" />
       <mass value="0.3000000119" />
@@ -902,5 +901,5 @@
     <visual>
       <material name="lidar-darkgrey" />
-      <origin rpy="${pi} 0.0000000000 0.0000000000"
+      <origin rpy="0.0000000000 0.0000000000 0.0000000000"
         xyz="0.0000000000 -0.0000000000 0.0000000000" />
       <geometry>

Commit message: v0.22.2

File: packages/src/uwaba_prototype_description/urdf/uwaba_prototype.urdf.xacro (robot description, xacro)
@@ -211,5 +211,5 @@
   </joint>
   <joint name="imu_base_joint" type="fixed">
-    <origin rpy="0.0000000000 0.0000000000 0.0000000000"
+    <origin rpy="0.0000000000 0.0000000000 ${pi/2}"
       xyz="0.061 -0.004 0.001875" />
     <parent link="base_link" />
@@ -845,5 +845,5 @@
   <link name="imu_frame">
     <collision name="imu_collision">
-      <origin rpy="0.0000000000 0.0000000000 0.0000000000"
+      <origin rpy="0.0000000000 0.0000000000 ${pi/2}"
         xyz="0 0 0" />
       <geometry>
@@ -853,5 +853,5 @@
     <visual>
       <!-- <material name="base-blue" /> -->
-      <origin rpy="0.0000000000 0.0000000000 0.0000000000"
+      <origin rpy="0.0000000000 0.0000000000 ${pi/2}"
         xyz="0 0 0" />
       <geometry>

Commit message: v0.23.2

File: packages/src/uwaba_prototype_description/urdf/uwaba_prototype.urdf.xacro (robot description, xacro)
@@ -211,5 +211,5 @@
   </joint>
   <joint name="imu_base_joint" type="fixed">
-    <origin rpy="0.0000000000 0.0000000000 ${pi/2}"
+    <origin rpy="0.0000000000 0.0000000000 ${-pi/2}"
       xyz="0.061 -0.004 0.001875" />
     <parent link="base_link" />
@@ -845,5 +845,5 @@
   <link name="imu_frame">
     <collision name="imu_collision">
-      <origin rpy="0.0000000000 0.0000000000 ${pi/2}"
+      <origin rpy="0.0000000000 0.0000000000 ${-pi/2}"
         xyz="0 0 0" />
       <geometry>
@@ -853,5 +853,5 @@
     <visual>
       <!-- <material name="base-blue" /> -->
-      <origin rpy="0.0000000000 0.0000000000 ${pi/2}"
+      <origin rpy="0.0000000000 0.0000000000 ${-pi/2}"
         xyz="0 0 0" />
       <geometry>

Commit message: v0.24.0

File: packages/src/uwaba_prototype_description/urdf/uwaba_prototype.urdf.xacro (robot description, xacro)
@@ -492,5 +492,5 @@
         xyz="-0.0000000075 0.0000000000 -0.0000000037" />
       <geometry>
-        <cylinder radius="0.0161000043" length="0.0219299998" />
+        <cylinder radius="0.0165" length="0.0219299998" />
       </geometry>
     </collision>
@@ -507,5 +507,5 @@
         xyz="-0.0000000075 0.0000000000 -0.0000000037" />
       <geometry>
-        <cylinder radius="0.0161000006" length="0.0219299980" />
+        <cylinder radius="0.0165" length="0.0219299980" />
       </geometry>
     </visual>
@@ -516,5 +516,5 @@
         xyz="0.0000000149 0.0000000000 -0.0000000075" />
       <geometry>
-        <cylinder radius="0.0161000025" length="0.0219299998" />
+        <cylinder radius="0.0165" length="0.0219299998" />
       </geometry>
     </collision>
@@ -531,5 +531,5 @@
         xyz="0.0000000149 0.0000000000 -0.0000000075" />
       <geometry>
-        <cylinder radius="0.0161000006" length="0.0219299980" />
+        <cylinder radius="0.0165" length="0.0219299980" />
       </geometry>
     </visual>
@@ -799,5 +799,5 @@
         xyz="0.0000000000 0.0000000000 0.0000000000" />
       <geometry>
-        <cylinder radius="0.0161000006" length="0.0219300017" />
+        <cylinder radius="0.0165" length="0.0219300017" />
       </geometry>
     </collision>
@@ -814,5 +814,5 @@
         xyz="0.0000000000 0.0000000000 0.0000000000" />
       <geometry>
-        <cylinder radius="0.0161000006" length="0.0219300017" />
+        <cylinder radius="0.0165" length="0.0219300017" />
       </geometry>
     </visual>
@@ -823,5 +823,5 @@
         xyz="0.0000000075 0.0000000075 0.0000000000" />
       <geometry>
-        <cylinder radius="0.0161000006" length="0.0219300017" />
+        <cylinder radius="0.0165" length="0.0219300017" />
       </geometry>
     </collision>
@@ -838,5 +838,5 @@
         xyz="0.0000000075 0.0000000075 0.0000000000" />
       <geometry>
-        <cylinder radius="0.0160999987" length="0.0219299998" />
+        <cylinder radius="0.0165" length="0.0219299998" />
       </geometry>
     </visual>

Commit message: Created filters for odom data

File: packages/src/uwaba_prototype_description/urdf/uwaba_prototype.urdf.xacro (robot description, xacro)
@@ -213,4 +213,5 @@
     <origin rpy="0.0000000000 0.0000000000 ${-pi/2}"
       xyz="0.061 -0.004 0.001875" />
+      <!-- xyz="0.061 -0.004 0.001875" -->
     <parent link="base_link" />
     <child link="imu_frame" />
@@ -218,5 +219,6 @@
   <joint name="laser_frame_base_joint" type="fixed">
     <origin rpy="${pi} 0.0000000000 0.0000000000"
-      xyz="-0.0110695819 -0.0000000043 0.0737789795" />
+      xyz="-0.024 0.0000000000 0.061" />
+      <!-- xyz="-0.0110695819 -0.0000000043 0.0737789795" -->
     <parent link="base_link" />
     <child link="laser_frame" />
@@ -845,5 +847,5 @@
   <link name="imu_frame">
     <collision name="imu_collision">
-      <origin rpy="0.0000000000 0.0000000000 ${-pi/2}"
+      <origin rpy="0.0000000000 0.0000000000 0.0000000000"
         xyz="0 0 0" />
       <geometry>
@@ -853,5 +855,5 @@
     <visual>
       <!-- <material name="base-blue" /> -->
-      <origin rpy="0.0000000000 0.0000000000 ${-pi/2}"
+      <origin rpy="0.0000000000 0.0000000000 0.0000000000"
         xyz="0 0 0" />
       <geometry>
